File: V1/V1.brd (EAGLE design)
At the start: 50 x 50 mm, 72 parts, among them Q1 MOSFET-NCHANNEL2N7002PW, Q2 MOSFET-NCHANNEL2N7002PW, U1 MCP2510SO, U2 MCP2561, U3 ATMEGA328P_TQFP, Y1 16MHz

Commit message: CHanged cap values on MCP2515 to 22pF
Parts:
- C3, C4: value 30pF -> 22pF
Changed lines of the file:
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@@
 <?xml version="1.0" encoding="utf-8"?>
 <!DOCTYPE eagle SYSTEM "eagle.dtd">
-<eagle version="7.4.0">
+<eagle version="7.6.0">
 <drawing>
 <settings>
@@
 <attribute name="VALUE" x="40.856" y="18.2235" size="1" layer="28" rot="MR180"/>
 </element>
-<element name="C3" library="adafruit" package="C0603K" value="30pF" x="8.509" y="20.574" smashed="yes">
+<element name="C3" library="adafruit" package="C0603K" value="22pF" x="8.509" y="20.574" smashed="yes">
 <attribute name="NAME" x="7.709" y="21.224" size="1" layer="25"/>
 </element>
-<element name="C4" library="adafruit" package="C0603K" value="30pF" x="2.7305" y="17.7165" smashed="yes" rot="MR0">
+<element name="C4" library="adafruit" package="C0603K" value="22pF" x="2.7305" y="17.7165" smashed="yes" rot="MR0">
 <attribute name="NAME" x="3.5305" y="18.3665" size="1" layer="26" rot="MR0"/>
 </element>

Commit message: update
Parts:
- R13, R14: value 100 -> 62
- R15, R16: value 1k -> 62
Changed lines of the file:
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@@
 <?xml version="1.0" encoding="utf-8"?>
 <!DOCTYPE eagle SYSTEM "eagle.dtd">
-<eagle version="7.6.0">
+<eagle version="7.4.0">
 <drawing>
 <settings>
@@
 <attribute name="NAME" x="30.226" y="11.1125" size="1" layer="26" font="vector" ratio="11" rot="MR0"/>
 </element>
-<element name="R13" library="SparkFun-Resistors" package="0603-RES" value="100" x="39.497" y="7.8105" smashed="yes">
+<element name="R13" library="SparkFun-Resistors" package="0603-RES" value="62" x="39.497" y="7.8105" smashed="yes">
 <attribute name="NAME" x="38.608" y="8.5725" size="1" layer="25" font="vector" ratio="11"/>
 <attribute name="VALUE" x="38.481" y="6.6675" size="1" layer="27" font="vector" ratio="11"/>
 </element>
-<element name="R14" library="SparkFun-Resistors" package="0603-RES" value="100" x="39.1795" y="11.2395" smashed="yes" rot="MR270">
+<element name="R14" library="SparkFun-Resistors" package="0603-RES" value="62" x="39.1795" y="11.2395" smashed="yes" rot="MR270">
 <attribute name="NAME" x="38.4175" y="12.1285" size="1" layer="26" font="vector" ratio="11" rot="MR270"/>
 <attribute name="VALUE" x="40.3225" y="12.2555" size="1" layer="28" font="vector" ratio="11" rot="MR270"/>
@@
 <attribute name="VALUE" x="41.3765" y="2.6045" size="1.016" layer="28" rot="MR0"/>
 </element>
-<element name="R15" library="SparkFun-Resistors" package="0603-RES" value="1k" x="7.4295" y="29.7815" rot="MR270"/>
-<element name="R16" library="SparkFun-Resistors" package="0603-RES" value="1k" x="14.0335" y="30.2895" rot="MR180"/>
+<element name="R15" library="SparkFun-Resistors" package="0603-RES" value="62" x="7.4295" y="29.7815" rot="MR270"/>
+<element name="R16" library="SparkFun-Resistors" package="0603-RES" value="62" x="14.0335" y="30.2895" rot="MR180"/>
 <element name="C18" library="adafruit" package="C0603K" value="4700pf" x="17.8435" y="29.5275" rot="MR270"/>
 </elements>
